File: 20180501 clock rgb.kicad_pcb (KiCad board)
At the start: 2 copper layers, 415 x 69 mm, 271 parts, among them J1 Barrel_Jack, J2 DB9M RS232, Q1 MMPQ2907A, Q2 MMPQ2907A, Q3 MMPQ2907A, SW1 SW_Push, SW2 SW_Push, SW3 SW_Push, SW4 SW_Push, SW5 SW_Push, SW6 SW_Push, U1 ATMEGA328P-PU, U10 MAX202, U2 74164, U3 74164, U5 LM7805_TO220, U6 PCA8856B, U7 PCA8856B, U8 DS3231-8, U9 LM7812_TO220, Y1 16MHz

Commit message: asdf
asd
Parts:
- added REF**: MountingHole_4mm, MountingHole:MountingHole_4mm, F.Cu at (22.0, 174.5)
- added REF**: MountingHole_4mm, MountingHole:MountingHole_4mm, F.Cu at (22.0, 235.5)
- added REF**: MountingHole_4mm, MountingHole:MountingHole_4mm, F.Cu at (429.0, 174.5)
- added REF**: MountingHole_4mm, MountingHole:MountingHole_4mm, F.Cu at (429.0, 235.5)
- D1, D14, D21: value APFA3010 -> LED_ARGB; footprint LED_SMD:LED_Avago_PLCC4_3.2x2.8mm_CW -> LED_SMD:LED_SK6812MINI_PLCC4_3.5x3.5mm_P1.75mm
- D10, D11, D12, D13, D15, D16, D17, D18, D19, D2, D20, D22, D23, D24, D25, D26, D27, D28, D29, D3, D30, D31, D32, D33, D34, D35, D36, D37, D38, D39, D4, D40, D41, D42, D43, D44, D45, D46, D47, D48, D49, D5, D50, D51, D52, D53, D54, D55, D56, D57, D58, D59, D6, D60, D61, D62, D63, D64, D65, D66, D67, D68, D69, D7, D70, D71, D72, D73, D74, D75, D76, D77, D78, D79, D8, D82, D83, D84, D85, D86, D87, D88, D9, D91, D92, D93, D94, D95, D96, D97: footprint LED_SMD:LED_Avago_PLCC4_3.2x2.8mm_CW -> LED_SMD:LED_SK6812MINI_PLCC4_3.5x3.5mm_P1.75mm
- turned D1 to 0 degrees
- turned D10 to 0 degrees
- turned D11 to 0 degrees
- turned D12 to 0 degrees
- turned D13 to 0 degrees
- turned D14 to 0 degrees
- turned D15 to 0 degrees
- turned D16 to 0 degrees
- turned D17 to 0 degrees
- turned D18 to 0 degrees
- turned D19 to 0 degrees
- turned D2 to 0 degrees
- turned D20 to 0 degrees
- turned D21 to 0 degrees
- turned D22 to 0 degrees
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Connections:
- D1 pad 1: /R -> Net-(D1-Pad1)
- D1 pad 2: Net-(D1-Pad2) -> /R
- D10 pad 1: /R -> Net-(D1-Pad1)
- D10 pad 2: Net-(D1-Pad2) -> /R
- D11 pad 1: /R -> Net-(D1-Pad1)
- D11 pad 2: Net-(D1-Pad2) -> /R
- D12 pad 1: /R -> Net-(D1-Pad1)
- D12 pad 2: Net-(D1-Pad2) -> /R
- D13 pad 1: /R -> Net-(D1-Pad1)
- D13 pad 2: Net-(D1-Pad2) -> /R
- D14 pad 1: /R -> Net-(D1-Pad1)
- D14 pad 2: Net-(D1-Pad2) -> /R
- D15 pad 1: /R -> Net-(D1-Pad1)
- D15 pad 2: Net-(D1-Pad2) -> /R
- D16 pad 1: /R -> Net-(D1-Pad1)
- D16 pad 2: Net-(D1-Pad2) -> /R
- D17 pad 1: /R -> Net-(D1-Pad1)
- D17 pad 2: Net-(D1-Pad2) -> /R
- D18 pad 1: /R -> Net-(D1-Pad1)
- D18 pad 2: Net-(D1-Pad2) -> /R
- D19 pad 1: /R -> Net-(D1-Pad1)
- D19 pad 2: Net-(D1-Pad2) -> /R
- D2 pad 1: /R -> Net-(D1-Pad1)
- D2 pad 2: Net-(D1-Pad2) -> /R
- D20 pad 1: /R -> Net-(D1-Pad1)
- D20 pad 2: Net-(D1-Pad2) -> /R
- D21 pad 1: /R -> Net-(D1-Pad1)
- D21 pad 2: Net-(D1-Pad2) -> /R
- D22 pad 1: /R -> Net-(D22-Pad1)
- D22 pad 2: Net-(D22-Pad2) -> /R
- D23 pad 1: /R -> Net-(D22-Pad1)
- D23 pad 2: Net-(D22-Pad2) -> /R
- D24 pad 1: /R -> Net-(D22-Pad1)
- D24 pad 2: Net-(D22-Pad2) -> /R
- D25 pad 1: /R -> Net-(D22-Pad1)
- D25 pad 2: Net-(D22-Pad2) -> /R
- D26 pad 1: /R -> Net-(D22-Pad1)
- D26 pad 2: Net-(D22-Pad2) -> /R
- D27 pad 1: /R -> Net-(D22-Pad1)
- D27 pad 2: Net-(D22-Pad2) -> /R
- D28 pad 1: /R -> Net-(D22-Pad1)
- D28 pad 2: Net-(D22-Pad2) -> /R
- D29 pad 1: /R -> Net-(D22-Pad1)
- D29 pad 2: Net-(D22-Pad2) -> /R
- D3 pad 1: /R -> Net-(D1-Pad1)
- D3 pad 2: Net-(D1-Pad2) -> /R
- D30 pad 1: /R -> Net-(D22-Pad1)
- D30 pad 2: Net-(D22-Pad2) -> /R
- D31 pad 1: /R -> Net-(D22-Pad1)
- D31 pad 2: Net-(D22-Pad2) -> /R
- D32 pad 1: /R -> Net-(D22-Pad1)
- D32 pad 2: Net-(D22-Pad2) -> /R
- D33 pad 1: /R -> Net-(D22-Pad1)
- D33 pad 2: Net-(D22-Pad2) -> /R
- D34 pad 1: /R -> Net-(D22-Pad1)
- D34 pad 2: Net-(D22-Pad2) -> /R
- D35 pad 1: /R -> Net-(D22-Pad1)
- D35 pad 2: Net-(D22-Pad2) -> /R
- D36 pad 1: /R -> Net-(D22-Pad1)
- D36 pad 2: Net-(D22-Pad2) -> /R
- D37 pad 1: /R -> Net-(D22-Pad1)
- D37 pad 2: Net-(D22-Pad2) -> /R
- D38 pad 1: /R -> Net-(D22-Pad1)
- D38 pad 2: Net-(D22-Pad2) -> /R
- D39 pad 1: /R -> Net-(D22-Pad1)
- D39 pad 2: Net-(D22-Pad2) -> /R
- D4 pad 1: /R -> Net-(D1-Pad1)
- D4 pad 2: Net-(D1-Pad2) -> /R
- D40 pad 1: /R -> Net-(D22-Pad1)
- D40 pad 2: Net-(D22-Pad2) -> /R
- D41 pad 1: /R -> Net-(D22-Pad1)
- D41 pad 2: Net-(D22-Pad2) -> /R
- D42 pad 1: /R -> Net-(D22-Pad1)
- D42 pad 2: Net-(D22-Pad2) -> /R
- D43 pad 1: /R -> +12V
- D43 pad 2: +12V -> /R
- D44 pad 1: /R -> +12V
- D44 pad 2: +12V -> /R
- D45 pad 1: /R -> Net-(D45-Pad1)
- D45 pad 2: Net-(D45-Pad2) -> /R
- D46 pad 1: /R -> Net-(D45-Pad1)
- D46 pad 2: Net-(D45-Pad2) -> /R
- D47 pad 1: /R -> Net-(D45-Pad1)
- D47 pad 2: Net-(D45-Pad2) -> /R
- D48 pad 1: /R -> Net-(D45-Pad1)
- D48 pad 2: Net-(D45-Pad2) -> /R
- D49 pad 1: /R -> Net-(D45-Pad1)
- D49 pad 2: Net-(D45-Pad2) -> /R
- D5 pad 1: /R -> Net-(D1-Pad1)
- D5 pad 2: Net-(D1-Pad2) -> /R
- D50 pad 1: /R -> Net-(D45-Pad1)
- D50 pad 2: Net-(D45-Pad2) -> /R
- D51 pad 1: /R -> Net-(D45-Pad1)
- D51 pad 2: Net-(D45-Pad2) -> /R
- D52 pad 1: /R -> Net-(D45-Pad1)
- D52 pad 2: Net-(D45-Pad2) -> /R
- D53 pad 1: /R -> Net-(D45-Pad1)
- D53 pad 2: Net-(D45-Pad2) -> /R
- D54 pad 1: /R -> Net-(D45-Pad1)
- D54 pad 2: Net-(D45-Pad2) -> /R
- D55 pad 1: /R -> Net-(D45-Pad1)
- D55 pad 2: Net-(D45-Pad2) -> /R
- D56 pad 1: /R -> Net-(D45-Pad1)
- D56 pad 2: Net-(D45-Pad2) -> /R
- D57 pad 1: /R -> Net-(D45-Pad1)
- D57 pad 2: Net-(D45-Pad2) -> /R
- D58 pad 1: /R -> Net-(D45-Pad1)
- D58 pad 2: Net-(D45-Pad2) -> /R
- D59 pad 1: /R -> Net-(D45-Pad1)
- D59 pad 2: Net-(D45-Pad2) -> /R
- D6 pad 1: /R -> Net-(D1-Pad1)
- D6 pad 2: Net-(D1-Pad2) -> /R
- D60 pad 1: /R -> Net-(D45-Pad1)
- D60 pad 2: Net-(D45-Pad2) -> /R
- D61 pad 1: /R -> Net-(D45-Pad1)
- D61 pad 2: Net-(D45-Pad2) -> /R
- D62 pad 1: /R -> Net-(D45-Pad1)
- D62 pad 2: Net-(D45-Pad2) -> /R
- D63 pad 1: /R -> Net-(D45-Pad1)
- D63 pad 2: Net-(D45-Pad2) -> /R
- D64 pad 1: /R -> Net-(D45-Pad1)
- D64 pad 2: Net-(D45-Pad2) -> /R
- D65 pad 1: /R -> Net-(D45-Pad1)
- D65 pad 2: Net-(D45-Pad2) -> /R
- D66 pad 1: /R -> Net-(D66-Pad1)
- D66 pad 2: Net-(D66-Pad2) -> /R
- D67 pad 1: /R -> Net-(D66-Pad1)
- D67 pad 2: Net-(D66-Pad2) -> /R
- D68 pad 1: /R -> Net-(D66-Pad1)
- D68 pad 2: Net-(D66-Pad2) -> /R
- D69 pad 1: /R -> Net-(D66-Pad1)
- D69 pad 2: Net-(D66-Pad2) -> /R
- D7 pad 1: /R -> Net-(D1-Pad1)
- D7 pad 2: Net-(D1-Pad2) -> /R
- D70 pad 1: /R -> Net-(D66-Pad1)
- D70 pad 2: Net-(D66-Pad2) -> /R
- D71 pad 1: /R -> Net-(D66-Pad1)
- D71 pad 2: Net-(D66-Pad2) -> /R
- D72 pad 1: /R -> Net-(D66-Pad1)
- D72 pad 2: Net-(D66-Pad2) -> /R
- D73 pad 1: /R -> Net-(D66-Pad1)
- D73 pad 2: Net-(D66-Pad2) -> /R
- D74 pad 1: /R -> Net-(D66-Pad1)
- D74 pad 2: Net-(D66-Pad2) -> /R
- D75 pad 1: /R -> Net-(D66-Pad1)
- D75 pad 2: Net-(D66-Pad2) -> /R
- D76 pad 1: /R -> Net-(D66-Pad1)
- D76 pad 2: Net-(D66-Pad2) -> /R
- D77 pad 1: /R -> Net-(D66-Pad1)
- D77 pad 2: Net-(D66-Pad2) -> /R
- D78 pad 1: /R -> Net-(D66-Pad1)
- D78 pad 2: Net-(D66-Pad2) -> /R
- D79 pad 1: /R -> Net-(D66-Pad1)
- D79 pad 2: Net-(D66-Pad2) -> /R
- D8 pad 1: /R -> Net-(D1-Pad1)
- D8 pad 2: Net-(D1-Pad2) -> /R
- D82 pad 1: /R -> Net-(D66-Pad1)
- D82 pad 2: Net-(D66-Pad2) -> /R
- D83 pad 1: /R -> Net-(D66-Pad1)
- D83 pad 2: Net-(D66-Pad2) -> /R
- D84 pad 1: /R -> Net-(D66-Pad1)
- D84 pad 2: Net-(D66-Pad2) -> /R
- D85 pad 1: /R -> Net-(D66-Pad1)
- D85 pad 2: Net-(D66-Pad2) -> /R
- D86 pad 1: /R -> Net-(D66-Pad1)
- D86 pad 2: Net-(D66-Pad2) -> /R
- D87 pad 1: /R -> Net-(D66-Pad1)
- D87 pad 2: Net-(D66-Pad2) -> /R
- D88 pad 1: /R -> Net-(D66-Pad1)
- D88 pad 2: Net-(D66-Pad2) -> /R
- D9 pad 1: /R -> Net-(D1-Pad1)
- D9 pad 2: Net-(D1-Pad2) -> /R
- Q1 pad 1: Net-(D1-Pad2) -> Net-(D1-Pad1)
- Q1 pad 2: Net-(D1-Pad2) -> Net-(D1-Pad1)
- Q1 pad 3: Net-(D22-Pad2) -> Net-(D22-Pad1)
- Q1 pad 4: Net-(D22-Pad2) -> Net-(D22-Pad1)
- Q1 pad 5: Net-(D45-Pad2) -> Net-(D45-Pad1)
- Q1 pad 6: Net-(D45-Pad2) -> Net-(D45-Pad1)
- Q1 pad 7: Net-(D66-Pad2) -> Net-(D66-Pad1)
- Q1 pad 8: Net-(D66-Pad2) -> Net-(D66-Pad1)
- Q2 pad 3: Net-(D91-Pad2) -> Net-(D91-Pad1)
- Q2 pad 4: Net-(D91-Pad2) -> Net-(D91-Pad1)
- Q2 pad 5: Net-(D92-Pad2) -> Net-(D92-Pad1)
- Q2 pad 6: Net-(D92-Pad2) -> Net-(D92-Pad1)
- Q2 pad 7: Net-(D93-Pad2) -> Net-(D93-Pad1)
- Q2 pad 8: Net-(D93-Pad2) -> Net-(D93-Pad1)
- Q3 pad 1: Net-(D94-Pad2) -> Net-(D94-Pad1)
- Q3 pad 2: Net-(D94-Pad2) -> Net-(D94-Pad1)
- Q3 pad 3: Net-(D95-Pad2) -> Net-(D95-Pad1)
- Q3 pad 4: Net-(D95-Pad2) -> Net-(D95-Pad1)
- Q3 pad 5: Net-(D96-Pad2) -> Net-(D96-Pad1)
- Q3 pad 6: Net-(D96-Pad2) -> Net-(D96-Pad1)
- Q3 pad 7: Net-(D97-Pad2) -> Net-(D97-Pad1)
- Q3 pad 8: Net-(D97-Pad2) -> Net-(D97-Pad1)
- R111 pad 1: Net-(D91-Pad1) -> Net-(D91-Pad2)
- R114 pad 1: Net-(D92-Pad1) -> Net-(D92-Pad2)
- R117 pad 1: Net-(D93-Pad1) -> Net-(D93-Pad2)
- R120 pad 1: Net-(D94-Pad1) -> Net-(D94-Pad2)
- R123 pad 1: Net-(D95-Pad1) -> Net-(D95-Pad2)
- R126 pad 1: Net-(D96-Pad1) -> Net-(D96-Pad2)
- R129 pad 1: Net-(D97-Pad1) -> Net-(D97-Pad2)
Routing:
- net Net-(D66-Pad1): track 0.00 -> 754.3 mm, vias 0 -> 4
- net Net-(D1-Pad2): track 724.6 -> 0.00 mm
- net Net-(D1-Pad1): track 0.00 -> 719.3 mm
- net Net-(D45-Pad1): track 0.00 -> 657.2 mm, vias 0 -> 2
- net Net-(D22-Pad2): track 634.7 -> 0.00 mm
- net Net-(D22-Pad1): track 0.00 -> 630.2 mm
- net Net-(D45-Pad2): track 493.8 -> 0.00 mm
- net Net-(D66-Pad2): track 473.7 -> 0.00 mm, vias 3 -> 0
- net /R: track 2447.8 -> 2165.8 mm, vias 63 -> 12
- net /B: track 2138.2 -> 2036.6 mm, vias 18 -> 11
- net Net-(D97-Pad1): track 2.98 -> 69.4 mm
- net Net-(D97-Pad2): track 70.2 -> 8.06 mm
- net Net-(D96-Pad1): track 10.5 -> 61.6 mm
- net Net-(D96-Pad2): track 60.8 -> 12.6 mm, vias 0 -> 1
- net /G: track 2100.4 -> 2061.0 mm, vias 69 -> 12
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